Commit message: fixed camera orientation

File: src/edu-elfin_simulation/elfin/elfin_description/urdf/elfin3_camera.urdf.xacro (robot description, xacro)
@@ -7,5 +7,5 @@
   <xacro:include filename="$(find elfin_description)/urdf/_d435.urdf.xacro" />
   <xacro:sensor_d435 name="camera" parent="elfin_end_link">
-    <origin xyz="0.1 0.0 -0.03" rpy="0 ${-PI/2} 0"/>
+    <origin xyz="0.1 0.0 -0.03" rpy="${PI} ${-PI/2} 0"/>
   </xacro:sensor_d435>
   <link name="world"/>
